File: hardware/orangecrab_r0.2.1/IO.kicad_sch (KiCad schematic)
At the start: 37 parts, among them J1 Conn_01x12, J2 Conn_01x16, J3 USB_C_Receptacle_USB2.0, SW1 SW_Push, U9 74HC4067BQ

Commit message: all IO gone/cleaned
Parts:
- removed C28, C71: 100nF, gkl_dipol:C_0201_0603Metric, symbol Device:C
- removed C76: 10nF, gkl_dipol:C_0201_0603Metric, symbol Device:C
- removed D1: LED_ARGB, gkl_led:0404LED_RGB, symbol Device:LED_ARGB
- removed J1: Conn_01x12, gkl_conn:Feather_PinHeader_1x12, symbol Connector_Generic:Conn_01x12
- removed J2: Conn_01x16, gkl_conn:Feather_PinHeader_1x16, symbol Connector_Generic:Conn_01x16
- removed J3: USB_C_Receptacle_USB2.0, Connector_USB:USB_C_Receptacle_HRO_TYPE-C-31-M-12, symbol Connector:USB_C_Receptacle_USB2.0
- removed R14, R16, R46: 5.1k, gkl_dipol:R_0201_0603Metric, symbol Device:R
- removed R20, R22: 1.5k, gkl_dipol:R_0201_0603Metric, symbol Device:R
- removed R21, R29: 20R, gkl_dipol:R_0201_0603Metric, symbol Device:R
- removed R23, R4: 4.7k, gkl_dipol:R_0201_0603Metric, symbol Device:R
- removed R24: 3.57k, gkl_dipol:R_0201_0603Metric, symbol Device:R
- removed R3, R48, R49, R50, R51, R6: 51R, gkl_dipol:R_0201_0603Metric, symbol Device:R
- removed R32, R33, R44, R45: 10k, gkl_dipol:R_0201_0603Metric, symbol Device:R
- removed SW1: SW_Push, gkl_misc:PTS_810_SMT_Switch, symbol Switch:SW_Push
- removed TP26, TP27, TP29: SMD_TP, gkl_misc:TestPoint_Pad_D0.5mm, symbol Connector:TestPoint_Flag
- removed U9: 74HC4067BQ, Package_DFN_QFN:Texas_RGY_R-PVQFN-N24_EP2.05x3.1mm, symbol 74xx:CD74HC4067M
Connections:
- no-connect marks 2 -> 0
Other:
- note removed: "Feather I/O"
- note removed: "Onboard rails connected to the ADC"
- note removed: "RESET +3V3 AREF GND ANALOG 0 ANALOG 1 ANALOG 2 ANALOG 3 ANALOG 4 ANALOG 5 I/O - SCK I/O - MOSI I/O - MISO I/O - RX I/O - TX I/O"
- note removed: "USB input"
- note removed: "USER LEDS"
- note removed: "VBAT (3 - 4.2V) EN VBUS (4.5-5.5V) I/O I/O I/O I/O I/O I/O I/O I/O - SCL I/O - SDA"
