File: hardware/orangecrab_r0.2.1/SDMMC.kicad_sch (KiCad schematic)
At the start: 9 parts, among them J4 MicroSd

Commit message: all IO gone/cleaned
Parts:
- removed C29: 10uF, Capacitor_SMD:C_0402_1005Metric, symbol Device:C
- removed C70: 100nF, gkl_dipol:C_0201_0603Metric, symbol Device:C
- removed FB1: 600R, Inductor_SMD:L_0402_1005Metric, symbol Device:FerriteBead_Small
- removed J4: MicroSd, gkl_conn:molex_microsd_1040310811, symbol Connector_Generic_MountingPin:Conn_01x09_MountingPin
- removed R28, R40, R41, R42, R43: 10k, gkl_dipol:R_0201_0603Metric, symbol Device:R
Other:
- note removed: "DAT2 DAT3/CD CMD VDD CLK VSS DAT0 DAT1 DET"
