File: hardware/orangecrab_r0.2.1/OrangeCrab.kicad_pcb (KiCad board)
At the start: 6 copper layers, 50.8 x 22.9 mm, 163 parts, among them J1 Conn_01x12_Male, J2 Conn_01x16_Male, J3 USB_C_Receptacle_USB2.0, J4 MicroSd, J5 JST, J6 Conn_01x05_Male, SW1 SW_Push, U1 TLV62569DRL, U10 NCP115-2.5, U2 TLV62569DRL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

Commit message: fix symbol links // try pcb/sch align
Parts:
- removed G***: LOGO, logo
- removed G***: LOGO, gkl_logos:gsd_logo_small
- removed G***: LOGO, gkl_logos:oshw_small
- J1: value Conn_01x12_Male -> Conn_01x12
- J2: value Conn_01x16_Male -> Conn_01x16
- J6: value Conn_01x05_Male -> Conn_01x05
- turned FB1 to -90 degrees
Connections:
- C29 pad 2: Net-(C29-Pad2) -> Net-(J4-Pin_4)
- C70 pad 2: Net-(C29-Pad2) -> Net-(J4-Pin_4)
- D2 pad 4: Net-(D2-Pad4) -> unconnected-(D2-BK-Pad4)
- FB1 pad 1: Net-(C29-Pad2) -> P3.3V
- FB1 pad 2: P3.3V -> Net-(J4-Pin_4)
- J3 pad A8: Net-(J3-PadA8) -> unconnected-(J3-SBU1-PadA8)
- J3 pad B8: Net-(J3-PadB8) -> unconnected-(J3-SBU2-PadB8)
- J4 pad 4: Net-(C29-Pad2) -> Net-(J4-Pin_4)
- U1 pad 6: Net-(U1-Pad6) -> unconnected-(U1-NC-Pad6)
- U2 pad 6: Net-(U2-Pad6) -> unconnected-(U2-NC-Pad6)
- U3 pad A10: Net-(U3-PadA10) -> unconnected-(U3A-PT27B/PCLKC0_1-PadA10)
- U3 pad A11: Net-(U3-PadA11) -> unconnected-(U3A-PT27A/PCLKT0_1-PadA11)
- U3 pad B11: Net-(U3-PadB11) -> unconnected-(U3A-PT4A-PadB11)
- U3 pad C11: Net-(U3-PadC11) -> unconnected-(U3A-PT4B-PadC11)
- U3 pad H18: Net-(U3-PadH18) -> unconnected-(U3E-PL38D-PadH18)
- U3 pad R16: Net-(U3-PadR16) -> unconnected-(U3G-PB18A/WRITEN-PadR16)
- U3 pad U15: Net-(U3-PadU15) -> unconnected-(U3H-DONE-PadU15)
- U3 pad V11: Net-(U3-PadV11) -> unconnected-(U3H-RESERVED-PadV11)
- U3 pad V12: Net-(U3-PadV12) -> unconnected-(U3H-RESERVED-PadV12)
- U3 pad V16: Net-(U3-PadV16) -> unconnected-(U3H-INITN-PadV16)
- U3 pad V2: Net-(U3-PadV2) -> unconnected-(U3H-RESERVED-PadV2)
- U3 pad V3: Net-(U3-PadV3) -> unconnected-(U3H-RESERVED-PadV3)
- U7 pad 6: Net-(U7-Pad6) -> unconnected-(U7-NC-Pad6)
Routing:
- net Net-(J4-Pin_4): track 0.00 -> 15.2 mm, vias 0 -> 3
- net Net-(C29-Pad2): track 15.2 -> 0.00 mm, vias 3 -> 0
Other:
- net class DDR3_CTRL_LM1.0 removed
- net class DDR3_DQS0_LM1.0 removed
- net class DDR3_DQS1_LM1.0 removed
- net class DDR_CLK_LM1.0 removed
- net class Default removed

Commit message: all IO gone/cleaned
Parts:
- removed C12, C13, C77: 4.7uF, Capacitor_SMD:C_0402_1005Metric
- removed C28, C70, C71: 100nF, gkl_dipol:C_0201_0603Metric
- removed C29: 10uF, Capacitor_SMD:C_0402_1005Metric
- removed C76: 10nF, gkl_dipol:C_0201_0603Metric
- removed D1, D2: LED_ARGB, gkl_led:0404LED_RGB
- removed FB1: 600R, Inductor_SMD:L_0402_1005Metric
- removed FID1, FID2, FID3, FID4, FID5, FID6: Fiducial, Fiducial:Fiducial_0.75mm_Mask1.5mm
- removed H1, H2: MountingHole, MountingHole:MountingHole_2.2mm_M2_Pad
- removed H3, H4: MountingHole, MountingHole:MountingHole_2.1mm
- removed J1: Conn_01x12, gkl_conn:Feather_PinHeader_1x12
- removed J2: Conn_01x16, gkl_conn:Feather_PinHeader_1x16
- removed J3: USB_C_Receptacle_USB2.0, Connector_USB:USB_C_Receptacle_HRO_TYPE-C-31-M-12
- removed J4: MicroSd, gkl_conn:molex_microsd_1040310811
- removed J5: JST, gkl_conn:JST_PH_B2B-PH-SM4-TB_1x02-1MP_P2.00mm_Vertical
- removed R10: 56.2k, gkl_dipol:R_0201_0603Metric
- removed R11: 3.09k, gkl_dipol:R_0201_0603Metric
- removed R12: 4.32k, gkl_dipol:R_0201_0603Metric
- removed R14, R16, R46: 5.1k, gkl_dipol:R_0201_0603Metric
- removed R20, R22: 1.5k, gkl_dipol:R_0201_0603Metric
- removed R21, R29: 20R, gkl_dipol:R_0201_0603Metric
- removed R23, R4, R8: 4.7k, gkl_dipol:R_0201_0603Metric
- removed R24, R9: 3.57k, gkl_dipol:R_0201_0603Metric
- removed R26, R28, R32, R33, R40, R41, R42, R43, R44, R45, R7: 10k, gkl_dipol:R_0201_0603Metric
- removed R3, R48, R49, R50, R51, R6: 51R, gkl_dipol:R_0201_0603Metric
- removed SW1: SW_Push, gkl_misc:PTS_810_SMT_Switch
- removed TP26, TP27, TP29: SMD_TP, gkl_misc:TestPoint_Pad_D0.5mm
- removed U5: BQ24232, Package_DFN_QFN:QFN-16-1EP_3x3mm_P0.5mm_EP1.75x1.75mm
- removed U9: 74HC4067BQ, Package_DFN_QFN:Texas_RGY_R-PVQFN-N24_EP2.05x3.1mm
Connections:
- U3 pad A8: IO_11 -> unconnected-(U3B-PT35B/PCLKC1_0-PadA8)
- U3 pad B10: IO_5 -> unconnected-(U3A-PT29A/PCLKT0_0-PadB10)
- U3 pad B8: IO_10 -> unconnected-(U3B-PT67A-PadB8)
- U3 pad B9: IO_6 -> unconnected-(U3B-PT33A/PCLKT1_1-PadB9)
- U3 pad C10: IO_SDA -> unconnected-(U3A-PT29B/PCLKC0_0-PadC10)
- U3 pad C8: IO_9 -> unconnected-(U3B-PT67B-PadC8)
- U3 pad C9: IO_SCL -> unconnected-(U3B-PT33B/PCLKC1_1-PadC9)
- U3 pad F1: ADC_CTRL1 -> unconnected-(U3D-PR35C-PadF1)
- U3 pad F2: ADC_MUX2 -> unconnected-(U3D-PR32A-PadF2)
- U3 pad F3: ADC_MUX1 -> unconnected-(U3D-PR26D/PCLKC3_0-PadF3)
- U3 pad F4: ADC_MUX0 -> unconnected-(U3D-PR26C/PCLKT3_0-PadF4)
- U3 pad G1: ADC_CTRL0 -> unconnected-(U3D-PR32B-PadG1)
- U3 pad G3: ADC_SENSE_LO -> unconnected-(U3D-PR29B-PadG3)
- U3 pad G4: IO_A4 -> unconnected-(U3D-PR26B/PCLKC3_1-PadG4)
- U3 pad H1: ADC_MUX3 -> unconnected-(U3D-PR35D-PadH1)
- U3 pad H3: ADC_SENSE_HI -> unconnected-(U3D-PR29A/GR_PCLK3_0-PadH3)
- U3 pad H4: IO_A3 -> unconnected-(U3D-PR26A/PCLKT3_1-PadH4)
- U3 pad L4: IO_A0 -> unconnected-(U3D-PR38B-PadL4)
- U3 pad M18: IO_1 -> unconnected-(U3G-PB6B/D4/MOSI2/IO4-PadM18)
- U3 pad N15: IO_MISO -> unconnected-(U3G-PB4A/D7/IO7-PadN15)
- U3 pad N16: IO_MOSI -> unconnected-(U3G-PB4B/D6/IO6-PadN16)
- U3 pad N17: IO_0 -> unconnected-(U3G-PB6A/D5/MISO2/IO5-PadN17)
- U3 pad N3: IO_A1 -> unconnected-(U3D-PR38D-PadN3)
- U3 pad N4: IO_A2 -> unconnected-(U3D-PR38C-PadN4)
- U3 pad R17: IO_SCK -> unconnected-(U3G-PB13A/SN/CSN-PadR17)
- U3 pad T17: IO_A5 -> unconnected-(U3G-PB13B/CS1N-PadT17)
Routing:
- net GND: track 250.6 -> 166.7 mm, vias 141 -> 103
- net ADC_MUX1: track 42.1 -> 0.00 mm, vias 1 -> 0
- net SD0_DAT0: track 41.7 -> 0.00 mm, vias 2 -> 0
- net ADC_MUX0: track 41.2 -> 0.00 mm, vias 1 -> 0
- net LED_R: track 40.4 -> 0.00 mm, vias 2 -> 0
- net LED_B: track 39.4 -> 0.00 mm, vias 2 -> 0
- net SD0_DAT1: track 38.6 -> 0.00 mm, vias 2 -> 0
- net ADC_CTRL1: track 35.6 -> 0.00 mm, vias 1 -> 0
- net ADC_MUX3: track 34.5 -> 0.00 mm, vias 1 -> 0
- net USER_BUTTON: track 34.8 -> 0.57 mm, vias 2 -> 0
- net ADC_MUX2: track 33.3 -> 0.00 mm, vias 1 -> 0
- net PUSB_VBUS: track 33.3 -> 0.00 mm, vias 4 -> 0
- net /IO/_USB_D_P: track 30.1 -> 0.00 mm, vias 3 -> 0
- net /IO/_USB_D_N: track 29.9 -> 0.00 mm, vias 3 -> 0
- net SD0_CMD: track 29.7 -> 0.00 mm, vias 2 -> 0
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- removed copper zone on In3.Cu, net PUSB_VBUS
- removed copper zone on F.Cu, net VBATT
- removed copper zone on In3.Cu, net VBATT
Other:
- board text removed: "+"
- board text removed: "0"
- board text removed: "1"
- board text removed: "10"
- board text removed: "11"
- board text removed: "12"
- board text removed: "13"
- board text removed: "2020-07-18"
- board text removed: "3V3"
- board text removed: "5"
- board text removed: "6"
- board text removed: "9"
- board text removed: "A0"
- board text removed: "A1"
- board text removed: "A2"
- board text removed: "A3"
- board text removed: "A4"
- board text removed: "A5"
- board text removed: "AREF"
- board text removed: "CHG"
- board text removed: "D+"
- board text removed: "D-"
- board text removed: "EN"
- board text removed: "Edge Rail"
- board text removed: "MISO"
- board text removed: "MOSI"
- board text removed: "Plated Half-holes"
- board text removed: "RST"
- board text removed: "SCK"
- board text removed: "SCL"
- board text removed: "SDA"
- board text removed: "Suggested tab locations"
- board text removed: "VBAT"
- board text removed: "VUSB"
- board text removed: "^_^"
- board text removed: "btn0"
- board text removed: "r0.2.1"

Commit message: more gnd/via cleanup
Routing:
- net GND: track 166.7 -> 154.2 mm, vias 103 -> 102
Changed lines of the file:
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@@
   (via (at 171.25 108.800001) (size 0.3) (drill 0.15) (layers "F.Cu" "B.Cu") (net 1))
   (via (at 152.21 106.58) (size 0.3) (drill 0.15) (layers "F.Cu" "B.Cu") (net 1))
-  (via (at 157.95 108.07) (size 0.3) (drill 0.15) (layers "F.Cu" "B.Cu") (net 1))
   (via (at 155.28 110.89) (size 0.28) (drill 0.15) (layers "F.Cu" "B.Cu") (net 1))
   (via (at 178.527008 96.4) (size 0.3) (drill 0.15) (layers "F.Cu" "B.Cu") (net 1))
@@
   (via (at 158.7 98.907863) (size 0.3) (drill 0.15) (layers "F.Cu" "B.Cu") (net 1))
   (via (at 178.55 104.250001) (size 0.3) (drill 0.15) (layers "F.Cu" "B.Cu") (net 1))
-  (segment (start 160.31 105.805) (end 160.31 105.010001) (width 0.121) (layer "B.Cu") (net 1))
   (segment (start 162.5388 100.7275) (end 162.7039 100.8926) (width 0.15) (layer "B.Cu") (net 1))
   (segment (start 157.7407 101.4006) (end 157.7407 101.859301) (width 0.15) (layer "B.Cu") (net 1))
   (segment (start 158.21 97.225) (end 157.88 97.225) (width 0.15) (layer "B.Cu") (net 1))
   (segment (start 157.877862 98.907863) (end 157.7 98.907863) (width 0.2) (layer "B.Cu") (net 1))
-  (segment (start 156.01 109.46) (end 157.305 109.46) (width 0.15) (layer "B.Cu") (net 1))
   (segment (start 177.71 108.845) (end 177.255001 108.845) (width 0.25) (layer "B.Cu") (net 1))
   (segment (start 160.47 99.900001) (end 160.47 99.630001) (width 0.2) (layer "B.Cu") (net 1))
@@
   (segment (start 157.88 98.400001) (end 157.88 98.727863) (width 0.15) (layer "B.Cu") (net 1))
   (segment (start 163.175901 98.9241) (end 162.7 99.400001) (width 0.15) (layer "B.Cu") (net 1))
-  (segment (start 157.305 109.46) (end 157.555 109.71) (width 0.15) (layer "B.Cu") (net 1))
   (segment (start 171.34 108.890001) (end 171.25 108.800001) (width 0.25) (layer "B.Cu") (net 1))
   (segment (start 179.995 106.01) (end 179.995 106.555) (width 0.25) (layer "B.Cu") (net 1))
@@
   (segment (start 160.68 103.380001) (end 160.7 103.400001) (width 0.15) (layer "B.Cu") (net 1))
   (segment (start 170.857 96.1) (end 170.927 96.1) (width 0.121) (layer "B.Cu") (net 1))
-  (segment (start 160.385 106.205) (end 160.41 106.18) (width 0.121) (layer "B.Cu") (net 1))
   (segment (start 163.73 99.930001) (end 163.7 99.900001) (width 0.2) (layer "B.Cu") (net 1))
   (segment (start 177.255001 108.845) (end 177.1 109.000001) (width 0.25) (layer "B.Cu") (net 1))
-  (segment (start 160.31 105.010001) (end 160.2 104.900001) (width 0.121) (layer "B.Cu") (net 1))
   (segment (start 177.13 109.030001) (end 177.1 109.000001) (width 0.2) (layer "B.Cu") (net 1))
   (segment (start 178.94091 101.98891) (end 178.927 101.975) (width 0.15) (layer "B.Cu") (net 1))
@@
   (segment (start 160.17 104.870001) (end 160.2 104.900001) (width 0.2) (layer "B.Cu") (net 1))
   (segment (start 160.87 98.900001) (end 160.87 98.570001) (width 0.15) (layer "B.Cu") (net 1))
-  (segment (start 163.135 108.725) (end 158.605 108.725) (width 0.121) (layer "B.Cu") (net 1))
   (segment (start 163.209999 102.9) (end 162.7 102.9) (width 0.15) (layer "B.Cu") (net 1))
   (segment (start 162.371001 105.728984) (end 161.958983 105.728984) (width 0.2) (layer "B.Cu") (net 1))
@@
   (segment (start 162.371001 105.728984) (end 162.706739 105.393246) (width 0.2) (layer "B.Cu") (net 1))
   (segment (start 168.19 108.1) (end 167.66 108.63) (width 0.25) (layer "B.Cu") (net 1))
-  (segment (start 159.555 106.435) (end 159.685 106.305) (width 0.121) (layer "B.Cu") (net 1))
   (segment (start 163.902 96.51) (end 164.537 95.875) (width 0.121) (layer "B.Cu") (net 1))
   (segment (start 162.5388 100.5014) (end 162.5388 100.7275) (width 0.15) (layer "B.Cu") (net 1))
@@
   (segment (start 178.35 102.120001) (end 178.495001 101.975) (width 0.25) (layer "B.Cu") (net 1))
   (segment (start 163.71 103.400001) (end 163.209999 102.9) (width 0.15) (layer "B.Cu") (net 1))
-  (segment (start 160.055 106.335) (end 160.085 106.305) (width 0.121) (layer "B.Cu") (net 1))
-  (segment (start 160.555 106.375) (end 160.385 106.205) (width 0.121) (layer "B.Cu") (net 1))
   (segment (start 165.293 96.84) (end 164.962 96.84) (width 0.121) (layer "B.Cu") (net 1))
   (segment (start 174.242832 100.309168) (end 174.502 100.05) (width 0.25) (layer "B.Cu") (net 1))
-  (segment (start 159.555 106.915) (end 159.555 106.435) (width 0.121) (layer "B.Cu") (net 1))
   (segment (start 160.68 102.900001) (end 160.68 103.380001) (width 0.15) (layer "B.Cu") (net 1))
   (segment (start 161.2 101.130001) (end 161.43 101.130001) (width 0.15) (layer "B.Cu") (net 1))
   (segment (start 163.33 102.400001) (end 163.33 102.030001) (width 0.2) (layer "B.Cu") (net 1))
-  (segment (start 157.555 110.505) (end 157.555 109.71) (width 0.15) (layer "B.Cu") (net 1))
   (segment (start 164.8781 99.9528) (end 164.8781 99.7528) (width 0.15) (layer "B.Cu") (net 1))
   (segment (start 163.97 107.070001) (end 164.35 107.070001) (width 0.15) (layer "B.Cu") (net 1))
   (segment (start 162.78 104.850001) (end 162.78 105.150001) (width 0.2) (layer "B.Cu") (net 1))
   (segment (start 165.011098 98.914999) (end 164.871099 98.775) (width 0.15) (layer "B.Cu") (net 1))
-  (segment (start 159.555 107.165836) (end 158.650836 108.07) (width 0.121) (layer "B.Cu") (net 1))
   (segment (start 161.18 98.400001) (end 160.7 98.400001) (width 0.2) (layer "B.Cu") (net 1))
   (segment (start 161.43 101.130001) (end 161.7 101.400001) (width 0.15) (layer "B.Cu") (net 1))
@@
   (segment (start 160.42 101.120001) (end 160.7 101.400001) (width 0.15) (layer "B.Cu") (net 1))
   (segment (start 178.97 108.1) (end 178.55 108.1) (width 0.25) (layer "B.Cu") (net 1))
-  (segment (start 160.41 105.905) (end 160.31 105.805) (width 0.121) (layer "B.Cu") (net 1))
-  (segment (start 160.41 106.18) (end 160.41 105.905) (width 0.121) (layer "B.Cu") (net 1))
-  (segment (start 160.085 106.305) (end 160.285 106.305) (width 0.121) (layer "B.Cu") (net 1))
   (segment (start 171.34 109.29) (end 171.34 108.890001) (width 0.25) (layer "B.Cu") (net 1))
   (segment (start 157.202 103.4) (end 157.202 102.592) (width 0.15) (layer "B.Cu") (net 1))
@@
   (segment (start 177.78 102.120001) (end 178.35 102.120001) (width 0.25) (layer "B.Cu") (net 1))
   (segment (start 163.33 102.030001) (end 163.2 101.900001) (width 0.2) (layer "B.Cu") (net 1))
-  (segment (start 160.555 106.915) (end 160.555 106.375) (width 0.121) (layer "B.Cu") (net 1))
-  (segment (start 160.285 106.305) (end 160.385 106.205) (width 0.121) (layer "B.Cu") (net 1))
   (segment (start 162.8469 100.8926) (end 163.2 100.5395) (width 0.15) (layer "B.Cu") (net 1))
   (segment (start 178.785 99.4) (end 178.94 99.245) (width 0.25) (layer "B.Cu") (net 1))
   (segment (start 161.25 105.320001) (end 161.55 105.320001) (width 0.2) (layer "B.Cu") (net 1))
-  (segment (start 159.685 106.305) (end 160.085 106.305) (width 0.121) (layer "B.Cu") (net 1))
   (segment (start 167.95 108.92) (end 167.66 108.63) (width 0.25) (layer "B.Cu") (net 1))
   (segment (start 157.7407 101.4006) (end 157.7407 100.940701) (width 0.15) (layer "B.Cu") (net 1))
@@
   (segment (start 157.7407 100.940701) (end 157.7 100.900001) (width 0.15) (layer "B.Cu") (net 1))
   (segment (start 164.8781 99.7528) (end 165.011098 99.619802) (width 0.15) (layer "B.Cu") (net 1))
-  (segment (start 160.055 106.915) (end 160.055 106.335) (width 0.121) (layer "B.Cu") (net 1))
   (segment (start 157.7 100.900001) (end 157.7 100.41) (width 0.15) (layer "B.Cu") (net 1))
   (segment (start 168.85 108.92) (end 167.95 108.92) (width 0.25) (layer "B.Cu") (net 1))

Commit message: delete redundant sheets
Connections:
- U3 pad H2: IO_12 -> unconnected-(U3D-PR29D-PadH2)
- U3 pad J1: SD0_DAT0 -> unconnected-(U3D-PR35B/VREF1_3-PadJ1)
- U3 pad J2: IO_13 -> unconnected-(U3D-PR35A-PadJ2)
- U3 pad J3: LED_B -> unconnected-(U3D-PR29C/GR_PCLK3_1-PadJ3)
- U3 pad K1: SD0_CLK -> unconnected-(U3D-PR41D-PadK1)
- U3 pad K2: SD0_CMD -> unconnected-(U3D-PR44A-PadK2)
- U3 pad K3: SD0_DAT1 -> unconnected-(U3D-PR41C-PadK3)
- U3 pad K4: LED_R -> unconnected-(U3D-PR38A-PadK4)
- U3 pad L1: SD0_CD -> unconnected-(U3D-PR44B-PadL1)
- U3 pad L3: SD0_DAT2 -> unconnected-(U3D-PR41B-PadL3)
- U3 pad M1: SD0_DAT3 -> unconnected-(U3D-PR47C/LRC_GPLL0T_IN-PadM1)
- U3 pad M2: USB_D- -> unconnected-(U3D-PR44C-PadM2)
- U3 pad M3: LED_G -> unconnected-(U3D-PR41A-PadM3)
- U3 pad N1: USB_D+ -> unconnected-(U3D-PR47D/LRC_GPLL0C_IN-PadN1)
- U3 pad N2: USB_PULLUP -> unconnected-(U3D-PR44D-PadN2)
