File: hardware/orangecrab_r0.2.1/DECOUPLING.kicad_sch (KiCad schematic)
At the start: 24 parts

Commit message: add some LCSC part numbers, stock all important parts
Parts:
- C48, C49, C52, C53, C56, C58, C60, C62, C63, C66, C67, C74: lcsc# (none) -> C272853
- C50, C51, C54, C55, C57, C59, C61, C64, C65, C68, C69, C75: lcsc# (none) -> C467016
Changed lines of the file:
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@@
+      (effects (font (size 1.27 1.27)) hide)
+    )
+    (property "lcsc#" "C272853" (at 33.02 34.29 0)
       (effects (font (size 1.27 1.27)) hide)
     )
@@
       (effects (font (size 1.27 1.27)) hide)
     )
+    (property "lcsc#" "C467016" (at 38.1 34.29 0)
+      (effects (font (size 1.27 1.27)) hide)
+    )
     (pin "1")
     (pin "2")
@@
     )
     (property "PN_1" "CC0201KRX5R7BB103" (at 54.61 34.29 0)
+      (effects (font (size 1.27 1.27)) hide)
+    )
+    (property "lcsc#" "C272853" (at 54.61 34.29 0)
       (effects (font (size 1.27 1.27)) hide)
     )
@@
       (effects (font (size 1.27 1.27)) hide)
     )
+    (property "lcsc#" "C467016" (at 59.69 34.29 0)
+      (effects (font (size 1.27 1.27)) hide)
+    )
     (pin "1")
     (pin "2")
@@
     )
     (property "PN_1" "CC0201KRX5R7BB103" (at 76.2 34.29 0)
+      (effects (font (size 1.27 1.27)) hide)
+    )
+    (property "lcsc#" "C272853" (at 76.2 34.29 0)
       (effects (font (size 1.27 1.27)) hide)
     )
@@
       (effects (font (size 1.27 1.27)) hide)
     )
+    (property "lcsc#" "C467016" (at 81.28 34.29 0)
+      (effects (font (size 1.27 1.27)) hide)
+    )
     (pin "1")
     (pin "2")
@@
     )
     (property "PN_1" "CC0201KRX5R7BB103" (at 97.79 34.29 0)
+      (effects (font (size 1.27 1.27)) hide)
+    )
+    (property "lcsc#" "C272853" (at 97.79 34.29 0)
       (effects (font (size 1.27 1.27)) hide)
     )
@@
       (effects (font (size 1.27 1.27)) hide)
     )
+    (property "lcsc#" "C467016" (at 102.87 34.29 0)
+      (effects (font (size 1.27 1.27)) hide)
+    )
     (pin "1")
     (pin "2")
@@
     )
     (property "PN_1" "CC0201KRX5R7BB103" (at 118.11 34.29 0)
+      (effects (font (size 1.27 1.27)) hide)
+    )
+    (property "lcsc#" "C272853" (at 118.11 34.29 0)
       (effects (font (size 1.27 1.27)) hide)
     )
@@
       (effects (font (size 1.27 1.27)) hide)
     )
+    (property "lcsc#" "C467016" (at 123.19 34.29 0)
+      (effects (font (size 1.27 1.27)) hide)
+    )
     (pin "1")
     (pin "2")
@@
     )
     (property "PN_1" "CC0201KRX5R7BB103" (at 33.02 67.31 0)
+      (effects (font (size 1.27 1.27)) hide)
+    )
+    (property "lcsc#" "C272853" (at 33.02 67.31 0)
       (effects (font (size 1.27 1.27)) hide)
     )
@@
       (effects (font (size 1.27 1.27)) hide)
     )
+    (property "lcsc#" "C467016" (at 38.1 67.31 0)
+      (effects (font (size 1.27 1.27)) hide)
+    )
     (pin "1")
     (pin "2")
@@
     )
     (property "PN_1" "CC0201KRX5R7BB103" (at 54.61 67.31 0)
+      (effects (font (size 1.27 1.27)) hide)
+    )
+    (property "lcsc#" "C272853" (at 54.61 67.31 0)
       (effects (font (size 1.27 1.27)) hide)
     )
@@
       (effects (font (size 1.27 1.27)) hide)
     )
+    (property "lcsc#" "C467016" (at 59.69 67.31 0)
+      (effects (font (size 1.27 1.27)) hide)
+    )
     (pin "1")
     (pin "2")
@@
     )
     (property "PN_1" "CC0201KRX5R7BB103" (at 97.79 67.31 0)
+      (effects (font (size 1.27 1.27)) hide)
+    )
+    (property "lcsc#" "C272853" (at 97.79 67.31 0)
       (effects (font (size 1.27 1.27)) hide)
     )
@@
       (effects (font (size 1.27 1.27)) hide)
     )
+    (property "lcsc#" "C467016" (at 102.87 67.31 0)
+      (effects (font (size 1.27 1.27)) hide)
+    )
     (pin "1")
     (pin "2")
@@
     )
     (property "PN_1" "CC0201KRX5R7BB103" (at 119.38 67.31 0)
+      (effects (font (size 1.27 1.27)) hide)
+    )
+    (property "lcsc#" "C272853" (at 119.38 67.31 0)
       (effects (font (size 1.27 1.27)) hide)
     )
@@
       (effects (font (size 1.27 1.27)) hide)
     )
+    (property "lcsc#" "C467016" (at 124.46 67.31 0)
+      (effects (font (size 1.27 1.27)) hide)
+    )
     (pin "1")
     (pin "2")
@@
     )
     (property "PN_1" "CC0201KRX5R7BB103" (at 97.79 96.52 0)
+      (effects (font (size 1.27 1.27)) hide)
+    )
+    (property "lcsc#" "C272853" (at 97.79 96.52 0)
       (effects (font (size 1.27 1.27)) hide)
     )
@@
       (effects (font (size 1.27 1.27)) hide)
     )
+    (property "lcsc#" "C467016" (at 102.87 96.52 0)
+      (effects (font (size 1.27 1.27)) hide)
+    )
     (pin "1")
     (pin "2")
@@
     )
     (property "PN_1" "CC0201KRX5R7BB103" (at 119.38 96.52 0)
+      (effects (font (size 1.27 1.27)) hide)
+    )
+    (property "lcsc#" "C272853" (at 119.38 96.52 0)
       (effects (font (size 1.27 1.27)) hide)
     )
@@
       (effects (font (size 1.27 1.27)) hide)
     )
+    (property "lcsc#" "C467016" (at 124.46 96.52 0)
+      (effects (font (size 1.27 1.27)) hide)
+    )
     (pin "1")
     (pin "2")
@@
     )
     (property "PN_1" "CC0201KRX5R7BB103" (at 142.24 96.52 0)
+      (effects (font (size 1.27 1.27)) hide)
+    )
+    (property "lcsc#" "C272853" (at 142.24 96.52 0)
       (effects (font (size 1.27 1.27)) hide)
     )
@@
       (effects (font (size 1.27 1.27)) hide)
     )
+    (property "lcsc#" "C467016" (at 147.32 96.52 0)
+      (effects (font (size 1.27 1.27)) hide)
+    )
