File: hardware/orangecrab_r0.2.1/DRAM.kicad_sch (KiCad schematic)
At the start: 23 parts, among them U4 MT41K64M16TW-107_J-TR

Commit message: add some LCSC part numbers, stock all important parts
Parts:
- C2, C27, C30, C31, C32, C33: lcsc# (none) -> C467016
- C21, C22, C3, C34, C35, C36, C37: lcsc# (none) -> C325464
- C23, C24: lcsc# (none) -> C109448
- FB2, FB3: lcsc# (none) -> C87550
- U4: lcsc# (none) -> C75475
Changed lines of the file:
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@@
+      (effects (font (size 1.27 1.27)) hide)
+    )
+    (property "lcsc#" "C75475" (at 160.02 102.87 0)
       (effects (font (size 1.27 1.27)) hide)
     )
@@
       (effects (font (size 1.27 1.27)) hide)
     )
+    (property "lcsc#" "C325464" (at 171.45 54.61 0)
+      (effects (font (size 1.27 1.27)) hide)
+    )
     (pin "1")
     (pin "2")
@@
       (effects (font (size 1.27 1.27)) hide)
     )
+    (property "lcsc#" "C325464" (at 176.53 54.61 0)
+      (effects (font (size 1.27 1.27)) hide)
+    )
     (pin "1")
     (pin "2")
@@
       (effects (font (size 1.27 1.27)) hide)
     )
+    (property "lcsc#" "C467016" (at 148.59 54.61 0)
+      (effects (font (size 1.27 1.27)) hide)
+    )
     (pin "1")
     (pin "2")
@@
       (effects (font (size 1.27 1.27)) hide)
     )
+    (property "lcsc#" "C467016" (at 153.67 54.61 0)
+      (effects (font (size 1.27 1.27)) hide)
+    )
     (pin "1")
     (pin "2")
@@
       (effects (font (size 1.27 1.27)) hide)
     )
+    (property "lcsc#" "C325464" (at 171.45 35.56 0)
+      (effects (font (size 1.27 1.27)) hide)
+    )
     (pin "1")
     (pin "2")
@@
       (effects (font (size 1.27 1.27)) hide)
     )
+    (property "lcsc#" "C325464" (at 176.53 35.56 0)
+      (effects (font (size 1.27 1.27)) hide)
+    )
     (pin "1")
     (pin "2")
@@
       (effects (font (size 1.27 1.27)) hide)
     )
+    (property "lcsc#" "C467016" (at 148.59 35.56 0)
+      (effects (font (size 1.27 1.27)) hide)
+    )
     (pin "1")
     (pin "2")
@@
       (effects (font (size 1.27 1.27)) hide)
     )
+    (property "lcsc#" "C467016" (at 153.67 35.56 0)
+      (effects (font (size 1.27 1.27)) hide)
+    )
     (pin "1")
     (pin "2")
@@
       (effects (font (size 1.27 1.27)) hide)
     )
+    (property "lcsc#" "" (at 193.04 95.25 0)
+      (effects (font (size 1.27 1.27)) hide)
+    )
     (pin "1")
     (pin "2")
@@
       (effects (font (size 1.27 1.27)) hide)
     )
+    (property "lcsc#" "C325464" (at 214.63 54.61 0)
+      (effects (font (size 1.27 1.27)) hide)
+    )
     (pin "1")
     (pin "2")
@@
       (effects (font (size 1.27 1.27)) hide)
     )
+    (property "lcsc#" "C109448" (at 219.71 54.61 0)
+      (effects (font (size 1.27 1.27)) hide)
+    )
     (pin "1")
     (pin "2")
@@
       (effects (font (size 1.27 1.27)) hide)
     )
+    (property "lcsc#" "C87550" (at 224.79 48.26 0)
+      (effects (font (size 1.27 1.27)) hide)
+    )
     (pin "1")
     (pin "2")
@@
       (effects (font (size 1.27 1.27)) hide)
     )
+    (property "lcsc#" "C325464" (at 214.63 81.28 0)
+      (effects (font (size 1.27 1.27)) hide)
+    )
     (pin "1")
     (pin "2")
@@
       (effects (font (size 1.27 1.27)) hide)
     )
+    (property "lcsc#" "C109448" (at 219.71 81.28 0)
+      (effects (font (size 1.27 1.27)) hide)
+    )
     (pin "1")
     (pin "2")
@@
     )
     (property "PN_1" "MMZ1005S601ET000" (at 224.79 74.93 0)
+      (effects (font (size 1.27 1.27)) hide)
+    )
+    (property "lcsc#" "C87550" (at 224.79 74.93 0)
       (effects (font (size 1.27 1.27)) hide)
     )
@@
       (effects (font (size 1.27 1.27)) hide)
     )
+    (property "lcsc#" "C467016" (at 66.04 142.24 0)
+      (effects (font (size 1.27 1.27)) hide)
+    )
     (pin "1")
     (pin "2")
@@
       (effects (font (size 1.27 1.27)) hide)
     )
+    (property "lcsc#" "" (at 74.93 134.62 0)
+      (effects (font (size 1.27 1.27)) hide)
+    )
     (pin "1")
     (pin "2")
@@
       (effects (font (size 1.27 1.27)) hide)
     )
+    (property "lcsc#" "" (at 74.93 137.16 0)
+      (effects (font (size 1.27 1.27)) hide)
+    )
     (pin "1")
     (pin "2")
@@
       (effects (font (size 1.27 1.27)) hide)
     )
+    (property "lcsc#" "" (at 73.66 88.9 0)
+      (effects (font (size 1.27 1.27)) hide)
+    )
     (pin "1")
     (pin "2")
@@
     )
     (property "PN_1" "0201WMF1001TCE" (at 73.66 99.06 0)
+      (effects (font (size 1.27 1.27)) hide)
+    )
+    (property "lcsc#" "" (at 73.66 99.06 0)
       (effects (font (size 1.27 1.27)) hide)
     )
@@
       (effects (font (size 1.27 1.27)) hide)
     )
+    (property "lcsc#" "C325464" (at 90.17 99.06 0)
+      (effects (font (size 1.27 1.27)) hide)
+    )
     (pin "1")
     (pin "2")
@@
       (effects (font (size 1.27 1.27)) hide)
     )
+    (property "lcsc#" "C467016" (at 85.09 99.06 0)
+      (effects (font (size 1.27 1.27)) hide)
+    )
