File: hardware/orangecrab_r0.2.1/DRAM.kicad_sch (KiCad schematic)
At the start: 23 parts, among them U4 MT41K64M16TW-107_J-TR

Commit message: populate LCSC# for missing passives
Parts:
- R1, R2: lcsc# (none) -> C138165
- R13, R5: lcsc# (none) -> C163499
- R19: lcsc# (none) -> C114755
Changed lines of the file:
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@@
       (effects (font (size 1.27 1.27)) hide)
     )
-    (property "lcsc#" "" (at 193.04 95.25 0)
+    (property "lcsc#" "C114755" (at 193.04 95.25 0)
       (effects (font (size 1.27 1.27)) hide)
     )
@@
       (effects (font (size 1.27 1.27)) hide)
     )
-    (property "lcsc#" "" (at 74.93 134.62 0)
+    (property "lcsc#" "C163499" (at 74.93 134.62 0)
       (effects (font (size 1.27 1.27)) hide)
     )
@@
       (effects (font (size 1.27 1.27)) hide)
     )
-    (property "lcsc#" "" (at 74.93 137.16 0)
+    (property "lcsc#" "C163499" (at 74.93 137.16 0)
       (effects (font (size 1.27 1.27)) hide)
     )
@@
       (effects (font (size 1.27 1.27)) hide)
     )
-    (property "lcsc#" "" (at 73.66 88.9 0)
+    (property "lcsc#" "C138165" (at 73.66 88.9 0)
       (effects (font (size 1.27 1.27)) hide)
     )
@@
       (effects (font (size 1.27 1.27)) hide)
     )
-    (property "lcsc#" "" (at 73.66 99.06 0)
-      (effects (font (size 1.27 1.27)) hide)
-    )
+    (property "lcsc#" "C138165" (at 73.66 99.06 0)
+      (effects (font (size 1.27 1.27)) hide)
+    )
