File: hardware/orangecrab_r0.2.1/FPGA.kicad_sch (KiCad schematic)
At the start: 14 parts, among them J6 Conn_01x05, U3 LFE5U-25F-8MG285C, U6 W25Q128JVP

Commit message: all IO gone/cleaned
Connections:
- net ADC_CTRL0: no longer names the net of U3.G1 (PR32B)
- net ADC_CTRL1: no longer names the net of U3.F1 (PR35C)
- net ADC_MUX0: no longer names the net of U3.F4 (PR26C/PCLKT3_0)
- net ADC_MUX1: no longer names the net of U3.F3 (PR26D/PCLKC3_0)
- net ADC_MUX2: no longer names the net of U3.F2 (PR32A)
- net ADC_MUX3: no longer names the net of U3.H1 (PR35D)
- net ADC_SENSE_HI: no longer names the net of U3.H3 (PR29A/GR_PCLK3_0)
- net ADC_SENSE_LO: no longer names the net of U3.G3 (PR29B)
- net IO_0: no longer names the net of U3.N17 (PB6A/D5/MISO2/IO5)
- net IO_1: no longer names the net of U3.M18 (PB6B/D4/MOSI2/IO4)
- net IO_10: no longer names the net of U3.B8 (PT67A)
- net IO_11: no longer names the net of U3.A8 (PT35B/PCLKC1_0)
- net IO_5: no longer names the net of U3.B10 (PT29A/PCLKT0_0)
- net IO_6: no longer names the net of U3.B9 (PT33A/PCLKT1_1)
- net IO_9: no longer names the net of U3.C8 (PT67B)
- net IO_A0: no longer names the net of U3.L4 (PR38B)
- net IO_A1: no longer names the net of U3.N3 (PR38D)
- net IO_A2: no longer names the net of U3.N4 (PR38C)
- net IO_A3: no longer names the net of U3.H4 (PR26A/PCLKT3_1)
- net IO_A4: no longer names the net of U3.G4 (PR26B/PCLKC3_1)
- net IO_A5: no longer names the net of U3.T17 (PB13B/CS1N)
- net IO_MISO: no longer names the net of U3.N15 (PB4A/D7/IO7)
- net IO_MOSI: no longer names the net of U3.N16 (PB4B/D6/IO6)
- net IO_SCK: no longer names the net of U3.R17 (PB13A/SN/CSN)
- net IO_SCL: no longer names the net of U3.C9 (PT33B/PCLKC1_1)
- net IO_SDA: no longer names the net of U3.C10 (PT29B/PCLKC0_0)
Changed lines of the file:
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@@
-    )
-  )
-  (global_label "IO_SCK" (shape input) (at 236.22 49.53 0)
-    (effects (font (size 1.524 1.524)) (justify left))
-    (property "Intersheetrefs" "${INTERSHEET_REFS}" (at 236.22 49.53 0)
-      (effects (font (size 1.27 1.27)) hide)
     )
   )
@@
     )
   )
-  (global_label "IO_A4" (shape input) (at 144.78 121.92 0)
-    (effects (font (size 1.27 1.27)) (justify left))
-    (property "Intersheetrefs" "${INTERSHEET_REFS}" (at 144.78 121.92 0)
-      (effects (font (size 1.27 1.27)) hide)
-    )
-  )
   (global_label "RAM_UDQS+" (shape input) (at 50.8 125.73 0)
     (effects (font (size 1.27 1.27)) (justify left))
@@
     )
   )
-  (global_label "IO_0" (shape input) (at 236.22 34.29 0)
-    (effects (font (size 1.524 1.524)) (justify left))
-    (property "Intersheetrefs" "${INTERSHEET_REFS}" (at 236.22 34.29 0)
-      (effects (font (size 1.27 1.27)) hide)
-    )
-  )
   (global_label "SD0_CMD" (shape input) (at 144.78 175.26 0)
     (effects (font (size 1.27 1.27)) (justify left))
@@
     )
   )
-  (global_label "ADC_MUX2" (shape input) (at 144.78 139.7 0)
-    (effects (font (size 1.27 1.27)) (justify left))
-    (property "Intersheetrefs" "${INTERSHEET_REFS}" (at 144.78 139.7 0)
-      (effects (font (size 1.27 1.27)) hide)
-    )
-  )
   (global_label "SD0_DAT2" (shape input) (at 144.78 167.64 0)
     (effects (font (size 1.27 1.27)) (justify left))
@@
     )
   )
-  (global_label "IO_SDA" (shape input) (at 49.53 184.15 0)
-    (effects (font (size 1.27 1.27)) (justify left))
-    (property "Intersheetrefs" "${INTERSHEET_REFS}" (at 49.53 184.15 0)
-      (effects (font (size 1.27 1.27)) hide)
-    )
-  )
   (global_label "RAM_ODT" (shape input) (at 50.8 107.95 0)
     (effects (font (size 1.27 1.27)) (justify left))
@@
     )
   )
-  (global_label "ADC_MUX3" (shape input) (at 144.78 152.4 0)
-    (effects (font (size 1.27 1.27)) (justify left))
-    (property "Intersheetrefs" "${INTERSHEET_REFS}" (at 144.78 152.4 0)
-      (effects (font (size 1.27 1.27)) hide)
-    )
-  )
   (global_label "RAM_LDM" (shape input) (at 118.11 50.8 0)
     (effects (font (size 1.27 1.27)) (justify left))
     (property "Intersheetrefs" "${INTERSHEET_REFS}" (at 118.11 50.8 0)
-      (effects (font (size 1.27 1.27)) hide)
-    )
-  )
-  (global_label "IO_A5" (shape input) (at 236.22 52.07 0)
-    (effects (font (size 1.27 1.27)) (justify left))
-    (property "Intersheetrefs" "${INTERSHEET_REFS}" (at 236.22 52.07 0)
       (effects (font (size 1.27 1.27)) hide)
     )
@@
     )
   )
-  (global_label "ADC_SENSE_HI" (shape input) (at 144.78 129.54 0)
-    (effects (font (size 1.27 1.27)) (justify left))
-    (property "Intersheetrefs" "${INTERSHEET_REFS}" (at 144.78 129.54 0)
-      (effects (font (size 1.27 1.27)) hide)
-    )
-  )
   (global_label "RAM_A15" (shape input) (at 50.8 31.75 0)
     (effects (font (size 1.27 1.27)) (justify left))
@@
     )
   )
-  (global_label "ADC_CTRL1" (shape input) (at 144.78 149.86 0)
-    (effects (font (size 1.27 1.27)) (justify left))
-    (property "Intersheetrefs" "${INTERSHEET_REFS}" (at 144.78 149.86 0)
-      (effects (font (size 1.27 1.27)) hide)
-    )
-  )
   (global_label "RAM_BA0" (shape input) (at 50.8 36.83 0)
     (effects (font (size 1.27 1.27)) (justify left))
@@
     (effects (font (size 1.524 1.524)) (justify left))
     (property "Intersheetrefs" "${INTERSHEET_REFS}" (at 210.82 104.14 0)
-      (effects (font (size 1.27 1.27)) hide)
-    )
-  )
-  (global_label "IO_A1" (shape input) (at 144.78 162.56 0)
-    (effects (font (size 1.27 1.27)) (justify left))
-    (property "Intersheetrefs" "${INTERSHEET_REFS}" (at 144.78 162.56 0)
       (effects (font (size 1.27 1.27)) hide)
     )
@@
     )
   )
-  (global_label "IO_MISO" (shape input) (at 236.22 29.21 0)
-    (effects (font (size 1.524 1.524)) (justify left))
-    (property "Intersheetrefs" "${INTERSHEET_REFS}" (at 236.22 29.21 0)
-      (effects (font (size 1.27 1.27)) hide)
-    )
-  )
   (global_label "SPI_CONFIG_SS" (shape input) (at 236.22 54.61 0)
     (effects (font (size 1.524 1.524)) (justify left))
@@
     )
   )
-  (global_label "IO_5" (shape input) (at 49.53 181.61 0)
-    (effects (font (size 1.27 1.27)) (justify left))
-    (property "Intersheetrefs" "${INTERSHEET_REFS}" (at 49.53 181.61 0)
-      (effects (font (size 1.27 1.27)) hide)
-    )
-  )
   (global_label "RAM_A8" (shape input) (at 50.8 77.47 0)
     (effects (font (size 1.27 1.27)) (justify left))
@@
     )
   )
-  (global_label "ADC_SENSE_LO" (shape input) (at 144.78 132.08 0)
-    (effects (font (size 1.27 1.27)) (justify left))
-    (property "Intersheetrefs" "${INTERSHEET_REFS}" (at 144.78 132.08 0)
-      (effects (font (size 1.27 1.27)) hide)
-    )
-  )
   (global_label "RAM_D15" (shape input) (at 118.11 40.64 0)
     (effects (font (size 1.27 1.27)) (justify left))
@@
     (effects (font (size 1.27 1.27)) (justify left))
     (property "Intersheetrefs" "${INTERSHEET_REFS}" (at 50.8 59.69 0)
-      (effects (font (size 1.27 1.27)) hide)
-    )
-  )
-  (global_label "IO_1" (shape input) (at 236.22 36.83 0)
-    (effects (font (size 1.524 1.524)) (justify left))
-    (property "Intersheetrefs" "${INTERSHEET_REFS}" (at 236.22 36.83 0)
-      (effects (font (size 1.27 1.27)) hide)
-    )
-  )
-  (global_label "IO_9" (shape input) (at 88.9 184.15 0)
-    (effects (font (size 1.27 1.27)) (justify left))
-    (property "Intersheetrefs" "${INTERSHEET_REFS}" (at 88.9 184.15 0)
       (effects (font (size 1.27 1.27)) hide)
     )
@@
     )
   )
-  (global_label "IO_MOSI" (shape input) (at 236.22 31.75 0)
-    (effects (font (size 1.524 1.524)) (justify left))
-    (property "Intersheetrefs" "${INTERSHEET_REFS}" (at 236.22 31.75 0)
-      (effects (font (size 1.27 1.27)) hide)
-    )
-  )
   (global_label "QSPI_D2" (shape input) (at 236.22 41.91 0)
     (effects (font (size 1.524 1.524)) (justify left))
@@
     (effects (font (size 1.27 1.27)) (justify left))
     (property "Intersheetrefs" "${INTERSHEET_REFS}" (at 259.08 74.93 0)
-      (effects (font (size 1.27 1.27)) hide)
-    )
-  )
-  (global_label "ADC_MUX1" (shape input) (at 144.78 127 0)
-    (effects (font (size 1.27 1.27)) (justify left))
-    (property "Intersheetrefs" "${INTERSHEET_REFS}" (at 144.78 127 0)
       (effects (font (size 1.27 1.27)) hide)
     )
@@
     )
   )
-  (global_label "ADC_MUX0" (shape input) (at 144.78 124.46 0)
-    (effects (font (size 1.27 1.27)) (justify left))
-    (property "Intersheetrefs" "${INTERSHEET_REFS}" (at 144.78 124.46 0)
-      (effects (font (size 1.27 1.27)) hide)
-    )
-  )
-  (global_label "IO_10" (shape input) (at 88.9 181.61 0)
-    (effects (font (size 1.27 1.27)) (justify left))
-    (property "Intersheetrefs" "${INTERSHEET_REFS}" (at 88.9 181.61 0)
-      (effects (font (size 1.27 1.27)) hide)
-    )
-  )
-  (global_label "IO_A2" (shape input) (at 144.78 160.02 0)
-    (effects (font (size 1.27 1.27)) (justify left))
-    (property "Intersheetrefs" "${INTERSHEET_REFS}" (at 144.78 160.02 0)
-      (effects (font (size 1.27 1.27)) hide)
-    )
-  )
   (global_label "ECP5_VREF" (shape passive) (at 67.31 54.61 0)
     (effects (font (size 1.27 1.27)) (justify left))
@@
     )
   )
-  (global_label "IO_SCL" (shape input) (at 88.9 173.99 0)
-    (effects (font (size 1.27 1.27)) (justify left))
-    (property "Intersheetrefs" "${INTERSHEET_REFS}" (at 88.9 173.99 0)
-      (effects (font (size 1.27 1.27)) hide)
-    )
-  )
-  (global_label "IO_A3" (shape input) (at 144.78 119.38 0)
-    (effects (font (size 1.27 1.27)) (justify left))
-    (property "Intersheetrefs" "${INTERSHEET_REFS}" (at 144.78 119.38 0)
-      (effects (font (size 1.27 1.27)) hide)
-    )
-  )
-  (global_label "IO_6" (shape input) (at 88.9 171.45 0)
-    (effects (font (size 1.27 1.27)) (justify left))
-    (property "Intersheetrefs" "${INTERSHEET_REFS}" (at 88.9 171.45 0)
-      (effects (font (size 1.27 1.27)) hide)
-    )
-  )
   (global_label "LED_R" (shape input) (at 144.78 154.94 0)
     (effects (font (size 1.27 1.27)) (justify left))
@@
     )
   )
-  (global_label "IO_11" (shape input) (at 88.9 179.07 0)
-    (effects (font (size 1.27 1.27)) (justify left))
-    (property "Intersheetrefs" "${INTERSHEET_REFS}" (at 88.9 179.07 0)
-      (effects (font (size 1.27 1.27)) hide)
-    )
-  )
   (global_label "RAM_LDQS-" (shape input) (at 118.11 55.88 0)
     (effects (font (size 1.27 1.27)) (justify left))
@@
     )
   )
-  (global_label "IO_A0" (shape input) (at 144.78 157.48 0)
-    (effects (font (size 1.27 1.27)) (justify left))
-    (property "Intersheetrefs" "${INTERSHEET_REFS}" (at 144.78 157.48 0)
-      (effects (font (size 1.27 1.27)) hide)
-    )
-  )
   (global_label "IO_13" (shape input) (at 144.78 144.78 0)
     (effects (font (size 1.27 1.27)) (justify left))
@@
       (effects (font (size 1.27 1.27)) hide)
     )
-  )
-  (global_label "ADC_CTRL0" (shape input) (at 144.78 142.24 0)
-    (effects (font (size 1.27 1.27)) (justify left))
-    (property "Intersheetrefs" "${INTERSHEET_REFS}" (at 144.78 142.24 0)
-      (effects (font (size 1.27 1.27)) hide)
-    )
