File: hardware/orangecrab_r0.2.1/FPGA.kicad_sch (KiCad schematic)
At the start: 16 parts, among them J6 Conn_01x05, U3 LFE5U-25F-8MG285C, U6 W25Q128JVP

Commit message: add some LCSC part numbers, stock all important parts
Parts:
- C1, C19, C25: lcsc# (none) -> C272853
- C20, C26, C4: lcsc# (none) -> C467016
- OSC1: lcsc# (none) -> C669070
- U6: lcsc# (none) -> C190862
Changed lines of the file:
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@@
       (effects (font (size 1.27 1.27)) hide)
     )
+    (property "lcsc#" "" (at 49.53 171.45 0)
+      (effects (font (size 1.27 1.27)) hide)
+    )
     (pin "A10")
     (pin "A11")
@@
       (effects (font (size 1.27 1.27)) hide)
     )
+    (property "lcsc#" "" (at 95.25 171.45 0)
+      (effects (font (size 1.27 1.27)) hide)
+    )
     (pin "A10")
     (pin "A11")
@@
       (effects (font (size 1.27 1.27)) hide)
     )
+    (property "lcsc#" "" (at 50.8 31.75 0)
+      (effects (font (size 1.27 1.27)) hide)
+    )
     (pin "A10")
     (pin "A11")
@@
       (effects (font (size 1.27 1.27)) hide)
     )
+    (property "lcsc#" "" (at 144.78 119.38 0)
+      (effects (font (size 1.27 1.27)) hide)
+    )
     (pin "A10")
     (pin "A11")
@@
       (effects (font (size 1.27 1.27)) hide)
     )
+    (property "lcsc#" "" (at 118.11 33.02 0)
+      (effects (font (size 1.27 1.27)) hide)
+    )
     (pin "A10")
     (pin "A11")
@@
       (effects (font (size 1.27 1.27)) hide)
     )
+    (property "lcsc#" "" (at 50.8 97.79 0)
+      (effects (font (size 1.27 1.27)) hide)
+    )
     (pin "A10")
     (pin "A11")
@@
       (effects (font (size 1.27 1.27)) hide)
     )
+    (property "lcsc#" "" (at 236.22 29.21 0)
+      (effects (font (size 1.27 1.27)) hide)
+    )
     (pin "A10")
     (pin "A11")
@@
       (effects (font (size 1.27 1.27)) hide)
     )
+    (property "lcsc#" "" (at 198.12 78.74 0)
+      (effects (font (size 1.27 1.27)) hide)
+    )
     (pin "A10")
     (pin "A11")
@@
       (effects (font (size 1.27 1.27)) hide)
     )
+    (property "lcsc#" "" (at 256.54 147.32 0)
+      (effects (font (size 1.27 1.27)) hide)
+    )
     (pin "A10")
     (pin "A11")
@@
       (effects (font (size 1.27 1.27)) hide)
     )
+    (property "lcsc#" "" (at 209.55 111.76 0)
+      (effects (font (size 1.27 1.27)) hide)
+    )
     (pin "1")
     (pin "2")
@@
       (effects (font (size 1.27 1.27)) hide)
     )
+    (property "lcsc#" "C190862" (at 201.93 148.59 0)
+      (effects (font (size 1.27 1.27)) hide)
+    )
     (pin "1")
     (pin "2")
@@
       (effects (font (size 1.27 1.27)) hide)
     )
+    (property "lcsc#" "C272853" (at 68.58 121.92 0)
+      (effects (font (size 1.27 1.27)) hide)
+    )
     (pin "1")
     (pin "2")
@@
       (effects (font (size 1.27 1.27)) hide)
     )
+    (property "lcsc#" "C467016" (at 73.66 121.92 0)
+      (effects (font (size 1.27 1.27)) hide)
+    )
     (pin "1")
     (pin "2")
@@
       (effects (font (size 1.27 1.27)) hide)
     )
+    (property "lcsc#" "C272853" (at 68.58 63.5 0)
+      (effects (font (size 1.27 1.27)) hide)
+    )
     (pin "1")
     (pin "2")
@@
       (effects (font (size 1.27 1.27)) hide)
     )
+    (property "lcsc#" "C467016" (at 73.66 63.5 0)
+      (effects (font (size 1.27 1.27)) hide)
+    )
     (pin "1")
     (pin "2")
@@
       (effects (font (size 1.27 1.27)) hide)
     )
+    (property "lcsc#" "C669070" (at 248.92 76.2 0)
+      (effects (font (size 1.27 1.27)) hide)
+    )
     (pin "1")
     (pin "2")
@@
       (effects (font (size 1.27 1.27)) hide)
     )
+    (property "lcsc#" "C272853" (at 143.51 67.31 0)
+      (effects (font (size 1.27 1.27)) hide)
+    )
     (pin "1")
     (pin "2")
@@
       (effects (font (size 1.27 1.27)) hide)
     )
+    (property "lcsc#" "C467016" (at 148.59 67.31 0)
+      (effects (font (size 1.27 1.27)) hide)
+    )
     (pin "1")
     (pin "2")
@@
       (effects (font (size 1.27 1.27)) hide)
     )
+    (property "lcsc#" "" (at 201.93 73.66 0)
+      (effects (font (size 1.27 1.27)) hide)
+    )
     (pin "1")
     (pin "2")
@@
       (effects (font (size 1.27 1.27)) hide)
     )
+    (property "lcsc#" "" (at 185.42 135.89 0)
+      (effects (font (size 1.27 1.27)) hide)
+    )
     (pin "1")
     (pin "2")
@@
       (effects (font (size 1.27 1.27)) hide)
     )
+    (property "lcsc#" "" (at 217.17 88.9 0)
+      (effects (font (size 1.27 1.27)) hide)
+    )
     (pin "1")
     (pin "2")
@@
       (effects (font (size 1.27 1.27)) hide)
     )
+    (property "lcsc#" "" (at 144.272 102.87 0)
+      (effects (font (size 1.27 1.27)) hide)
+    )
     (pin "1")
     (instances
@@
       (effects (font (size 1.27 1.27)) hide)
     )
+    (property "lcsc#" "" (at 144.272 100.33 0)
+      (effects (font (size 1.27 1.27)) hide)
+    )
     (pin "1")
     (instances
@@
       (effects (font (size 1.27 1.27)) hide)
     )
+    (property "lcsc#" "" (at 264.16 95.25 0)
+      (effects (font (size 1.27 1.27)) hide)
+    )

Commit message: populate LCSC# for missing passives
Parts:
- R27, R30, R39: lcsc# (none) -> C138135
- R31: lcsc# (none) -> C155737
- U3: lcsc# (none) -> C000000
Changed lines of the file:
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@@
       (effects (font (size 1.27 1.27)) hide)
     )
-    (property "lcsc#" "" (at 49.53 171.45 0)
+    (property "lcsc#" "C000000" (at 49.53 171.45 0)
       (effects (font (size 1.27 1.27)) hide)
     )
@@
       (effects (font (size 1.27 1.27)) hide)
     )
-    (property "lcsc#" "" (at 95.25 171.45 0)
+    (property "lcsc#" "C000000" (at 95.25 171.45 0)
       (effects (font (size 1.27 1.27)) hide)
     )
@@
       (effects (font (size 1.27 1.27)) hide)
     )
-    (property "lcsc#" "" (at 50.8 31.75 0)
+    (property "lcsc#" "C000000" (at 50.8 31.75 0)
       (effects (font (size 1.27 1.27)) hide)
     )
@@
       (effects (font (size 1.27 1.27)) hide)
     )
-    (property "lcsc#" "" (at 144.78 119.38 0)
+    (property "lcsc#" "C000000" (at 144.78 119.38 0)
       (effects (font (size 1.27 1.27)) hide)
     )
@@
       (effects (font (size 1.27 1.27)) hide)
     )
-    (property "lcsc#" "" (at 118.11 33.02 0)
+    (property "lcsc#" "C000000" (at 118.11 33.02 0)
       (effects (font (size 1.27 1.27)) hide)
     )
@@
       (effects (font (size 1.27 1.27)) hide)
     )
-    (property "lcsc#" "" (at 50.8 97.79 0)
+    (property "lcsc#" "C000000" (at 50.8 97.79 0)
       (effects (font (size 1.27 1.27)) hide)
     )
@@
       (effects (font (size 1.27 1.27)) hide)
     )
-    (property "lcsc#" "" (at 236.22 29.21 0)
+    (property "lcsc#" "C000000" (at 236.22 29.21 0)
       (effects (font (size 1.27 1.27)) hide)
     )
@@
       (effects (font (size 1.27 1.27)) hide)
     )
-    (property "lcsc#" "" (at 198.12 78.74 0)
+    (property "lcsc#" "C000000" (at 198.12 78.74 0)
       (effects (font (size 1.27 1.27)) hide)
     )
@@
       (effects (font (size 1.27 1.27)) hide)
     )
-    (property "lcsc#" "" (at 256.54 147.32 0)
+    (property "lcsc#" "C000000" (at 256.54 147.32 0)
       (effects (font (size 1.27 1.27)) hide)
     )
@@
       (effects (font (size 1.27 1.27)) hide)
     )
-    (property "lcsc#" "" (at 209.55 111.76 0)
+    (property "lcsc#" "C138135" (at 209.55 111.76 0)
       (effects (font (size 1.27 1.27)) hide)
     )
@@
       (effects (font (size 1.27 1.27)) hide)
     )
-    (property "lcsc#" "" (at 201.93 73.66 0)
+    (property "lcsc#" "C155737" (at 201.93 73.66 0)
       (effects (font (size 1.27 1.27)) hide)
     )
@@
       (effects (font (size 1.27 1.27)) hide)
     )
-    (property "lcsc#" "" (at 185.42 135.89 0)
+    (property "lcsc#" "C138135" (at 185.42 135.89 0)
       (effects (font (size 1.27 1.27)) hide)
     )
@@
       (effects (font (size 1.27 1.27)) hide)
     )
-    (property "lcsc#" "" (at 217.17 88.9 0)
+    (property "lcsc#" "C138135" (at 217.17 88.9 0)
       (effects (font (size 1.27 1.27)) hide)
     )
